File: Projects/Project Name/Work/esempio1_git/esempio1_git.kicad_sch (KiCad schematic)
At the start: 4 parts

Commit message: Update 1
modificato formato foglio
Other:
- company: (none) -> Kineton Società Benefit S.r.l.
- title: (none) -> Esempio 1 git
Changed lines of the file:
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@@
 	(generator_version "8.0")
 	(paper "A4")
+	(title_block
+		(title "Esempio 1 git")
+		(date "2025-02-04")
+		(rev "rev01")
+		(company "Kineton Società Benefit S.r.l.")
+	)
 	(symbol
 		(lib_id "Device:R")

Commit message: Update 2
Aggiunta MCU
Parts:
- removed R1, R2, R3, R4: R, symbol Device:R
Other:
- added sheet BLOCK DIAGRAM (BLOCK DIAGRAM.kicad_sch)
- added sheet CAN (CAN.kicad_sch)
- added sheet FILTERS (FILTERS.kicad_sch)
- added sheet MCU (MCU.kicad_sch)
- added sheet MECHANICAL (MECHANICAL.kicad_sch)
- added sheet MOSFET DRIVER (MOSFET DRIVER.kicad_sch)
- added sheet MOSFETs (MOSFETs.kicad_sch)
- added sheet OVERVIEW (OVERVIEW.kicad_sch)
- title: Esempio 1 git -> Esempio 1 git - E-S-C
