File: Projects/Project Name/Work/esempio1_git/MOSFET DRIVER.kicad_sch (KiCad schematic)
At the start: 0 parts

Commit message: Update 2
Aggiunta MosfetDriver
Parts:
- added C18, C19, C21, C22, C25, C35: 2.2u, CRF1:SMD-0603_c, symbol BLDC_4-rescue:C-RESCUE-BLDC_4
- added C20: 120p, CRF1:SMD-0603_c, symbol BLDC_4-rescue:C-RESCUE-BLDC_4
- added C23: 6.8n, CRF1:SMD-0603_c, symbol BLDC_4-rescue:C-RESCUE-BLDC_4
- added C24: 22n, CRF1:SMD-0603_c, symbol BLDC_4-rescue:C-RESCUE-BLDC_4
- added C26, C27, C28, C37, C39, C40, C42, C43: 10u,50V, CRF1:SMD-1206, symbol BLDC_4-rescue:C-RESCUE-BLDC_4
- added C29: 100n, CRF1:SMD-0603_c, symbol BLDC_4-rescue:C-RESCUE-BLDC_4
- added C30, C31, C32: 220n, CRF1:SMD-0603_c, symbol BLDC_4-rescue:C-RESCUE-BLDC_4
- added C33, C34: 2.2n, CRF1:SMD-0603_c, symbol BLDC_4-rescue:C-RESCUE-BLDC_4
- added C36, C38: 100u, w_smd_cap:c_tant_B, symbol BLDC_4-rescue:CP1-RESCUE-BLDC_4
- added C41: 15u, 100v, w_smd_cap:c_2220, symbol BLDC_4-rescue:C-RESCUE-BLDC_4
- added C44: 15u,100V, w_smd_cap:c_2220, symbol BLDC_4-rescue:C-RESCUE-BLDC_4
- added D4: DIODESCH, Diodes_SMD:SMA_Handsoldering, symbol BLDC_4-rescue:DIODESCH
- added D5: TVS 5V, w_smd_diode:do214ac, symbol BLDC_4-rescue:DIODE
- added L1: 22u, w_smd_inductors:inductor_smd_8x5mm, symbol BLDC_4-rescue:INDUCTOR
- added R11: 18k, CRF1:SMD-0603_r, symbol BLDC_4-rescue:R-RESCUE-BLDC_4
- added R12: 3k3, CRF1:SMD-0603_r, symbol BLDC_4-rescue:R-RESCUE-BLDC_4
- added R13: 10k, CRF1:SMD-0603_r, symbol BLDC_4-rescue:R-RESCUE-BLDC_4
- added R14: 15k, CRF1:SMD-0603_r, symbol BLDC_4-rescue:R-RESCUE-BLDC_4
- added R15: 220k, CRF1:SMD-0603_r, symbol BLDC_4-rescue:R-RESCUE-BLDC_4
- added R16: 1M, CRF1:SMD-0603_r, symbol BLDC_4-rescue:R-RESCUE-BLDC_4
- added R17, R18, R19, R20: 100R, CRF1:SMD-0603_r, symbol BLDC_4-rescue:R-RESCUE-BLDC_4
- added R21, R23, R25: 39k, CRF1:SMD-0603_r, symbol BLDC_4-rescue:R-RESCUE-BLDC_4
- added R22, R24, R26: 2k2, CRF1:SMD-0603_r, symbol BLDC_4-rescue:R-RESCUE-BLDC_4
- added U2: DRV8302, CRF1:TSSOP-56-PP, symbol bldc:DRV8302
- added U3: TC2117, CRF1:SOT-223, symbol BLDC_4-rescue:NCP1117ST33T3G
Connections:
- new net: C29.1, D4.2 (K), L1.1, U2.50 (PH), U2.51 (PH)
- new net: C29.2, U2.52 (BST_BK)
- new net: C25.2, U2.27 (AVDD)
- new net: R15.2, U2.1 (RT_CLK)
- new net: C21.2, C22.2, U2.11 (OC_ADJ), U2.23 (DVDD)
- new net: C18.1, C19.1, U2.13 (GVDD)
- new net: C24.1, U2.14 (CP1)
- new net: C24.2, U2.15 (CP2)
- new net: C20.2, R14.2, U2.2 (COMP)
- new net: R11.2, R12.1, U2.3 (VSENSE)
- new net: C34.2, R20.2, U2.30 (SP2)
- new net: C34.1, R19.2, U2.31 (SN2)
- new net: C33.2, R18.2, U2.32 (SP1)
- new net: C33.1, R17.2, U2.33 (SN1)
- new net: C32.2, U2.38 (BST_C)
- new net: C31.2, U2.43 (BST_B)
- new net: C30.2, U2.48 (BST_A)
- new net: R16.2, U2.49 (BIAS)
- new net: R13.1, U2.7 (DTC)
- new net: C23.2, R14.1
- new net +5V: C38.1, D5.2 (K), L1.2, R11.1, U3.3 (VI)
- new net BR_SO1: U2.25 (SO1)
- new net BR_SO2: U2.26 (SO2)
- new net DC_CAL: U2.12 (DC_CAL)
- new net EN_GATE: U2.16 (EN_GATE)
- new net FAULT: U2.6 (FAULT)
- new net GND: C18.2, C19.2, C20.1, C21.1, C22.1, C23.1, C25.1, C26.2, C27.2, C28.2, C35.2, C36.2, C37.1, C38.2, C39.1, C40.1, C41.1, C42.1, C43.1, C44.1, D4.1 (A), D5.1 (A), R12.2, R13.2, R15.1, R16.1, R22.1, R24.1, R26.1, U2.10 (GAIN), U2.28 (AGND), U2.57 (GND(POWER_PAD)), U2.8 (M_PWM), U3.1 (GND)
- new net H1: U2.17 (INH_A)
- new net H1_LOW: U2.44 (SL_A)
- new net H1_VS: C30.1, R25.1, U2.46 (SH_A)
- new net H2: U2.19 (INH_B)
- new net H2_LOW: U2.39 (SL_B)
- new net H2_VS: C31.1, R23.1, U2.41 (SH_B)
- new net H3: U2.21 (INH_C)
- new net H3_LOW: U2.34 (SL_C)
- new net H3_VS: C32.1, R21.1, U2.36 (SH_C)
- new net L1: U2.18 (INL_A)
- new net L2: U2.20 (INL_B)
- new net L3: U2.22 (INL_C)
- new net M_H1: U2.47 (GH_A)
- new net M_H2: U2.42 (GH_B)
- new net M_H3: U2.37 (GH_C)
- new net M_L1: U2.45 (GL_A)
- new net M_L2: U2.40 (GL_B)
- new net M_L3: U2.35 (GL_C)
- new net SENS1: R21.2, R22.2
- new net SENS2: R23.2, R24.2
- new net SENS3: R25.2, R26.2
- new net SH1_A: R17.1
- new net SH1_B: R18.1
- new net SH2_A: R19.1
- new net SH2_B: R20.1
- new net VCC: C35.1, C36.1, U2.24 (REF), U2.9 (M_OC), U3.2 (VO)
- new net V_SUPPLY: C26.1, C27.1, C28.1, C37.2, C39.2, C40.2, C41.2, C42.2, C43.2, C44.2, U2.29 (PVDD1), U2.53 (PVDD2), U2.54 (PVDD2)
- no-connect marks 0 -> 4
Other:
- note added: "3.3v regulator for the logic"
- note added: "BULK CAPACITANCE KEEP AS CLOSE AS POSSIBLE TO THE IC AND TO THE DRIVER INPUT LOOP"
- note added: "MCU must sense the voltage at each phase"
